File: hardware/poeremote.sch (KiCad schematic (older format))
At the start: 106 parts, among them J1 3.3VDC, J3 RJ45, J4 SERIAL, J5 ISP, J7 LAMP, P1 CONN_5, P2 CONN_10, Q1 SOT23-BEC, Q2 PNP, Sw1 SPST-D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

Commit message: Updated to V2.2 board, including firmware. Still working on a bug or two, but it mostly works.
Parts:
- C1, C11, C3, C30: MPN C0805C106M9PACTU -> 08056D106MAT2A
- C12: MPN (none) -> C0603C102K1RACTU; Voltage 100 -> (none)
- C2: value 22uF -> 10uf; MPN (none) -> 08056D106MAT2A; Mouser Part Number 810-C1608X5R0J226M -> 603-CC603MRX5R5BB106; Supplier (none) -> Avnet
- C22: MPN C0603C332K5RACTU -> 06035C332KAT2A; Voltage 16 -> 16V
- C23: MPN C0603C332K5RACTU -> 06035C332KAT2A
- C27: value .1uF -> 100nF; MPN 12061C104KAT2A -> C0603C104K3RAC7411
- C28, C29: value 10-100nF -> 100nF; MPN 12061C104KAT2A -> C0603C104K3RAC7411
- C33: value .1uF -> 100nF
- C35: value 0.1uF -> 100nF; MPN 12061C104KAT2A -> C0603C104K3RAC7411
- L3: value FB -> 30ohmFB
- R17, R18, R19, R20, R21, R22, R23, R24, R25, R26, R27, R28, R29, R30, R31, R32: MPN (none) -> ERJ-3EKF51R0V; Supplier (none) -> Avnet
- X1: value 15MHz -> 25MHz
Changed lines of the file:
@@
-EESchema Schematic File Version 2  date Mon 18 Feb 2013 01:28:21 AM EST
+EESchema Schematic File Version 2  date Sun 24 Feb 2013 10:26:27 PM EST
 LIBS:power
 LIBS:device
@@
 Sheet 1 1
 Title ""
-Date "18 feb 2013"
+Date "25 feb 2013"
 Rev ""
 Comp ""
@@
 F 1 "10uf" H 20600 3900 50  0000 L CNN
 F 4 "603-CC603MRX5R5BB106" H 20550 4000 60  0001 C CNN "Mouser Part Number"
-F 5 "C0805C106M9PACTU" H 10300 3400 60  0001 C CNN "MPN"
+F 5 "08056D106MAT2A" H 10300 3400 60  0001 C CNN "MPN"
 F 6 "Avnet" H 10300 3400 60  0001 C CNN "Supplier"
 	1    20550 4000
@@
 F 1 "10uf" H 22100 3300 50  0000 L CNN
 F 4 "603-CC603MRX5R5BB106" H 22050 3400 60  0001 C CNN "Mouser Part Number"
-F 5 "C0805C106M9PACTU" H 10300 3400 60  0001 C CNN "MPN"
+F 5 "08056D106MAT2A" H 10300 3400 60  0001 C CNN "MPN"
 F 6 "Avnet" H 10300 3400 60  0001 C CNN "Supplier"
 	1    22050 3400
@@
 $EndComp
 $Comp
-L C C2
-U 1 1 4FF52DF5
-P 20200 2650
-F 0 "C2" H 20250 2750 50  0000 L CNN
-F 1 "22uF" H 20250 2550 50  0000 L CNN
-F 4 "810-C1608X5R0J226M" H 20200 2650 60  0001 C CNN "Mouser Part Number"
-	1    20200 2650
-	1    0    0    -1
-$EndComp
-$Comp
 L LM358 U1
 U 2 1 4FF52DC8
@@
 P 18400 900
 F 0 "C35" H 18450 1000 50  0000 L CNN
-F 1 "0.1uF" H 18450 800 50  0000 L CNN
+F 1 "100nF" H 18450 800 50  0000 L CNN
 F 4 "581-060316C104K" H 18400 900 60  0001 C CNN "Mouser Part Number"
-F 5 "12061C104KAT2A" H 2050 6700 60  0001 C CNN "MPN"
+F 5 "C0603C104K3RAC7411" H 2050 6700 60  0001 C CNN "MPN"
 F 6 "Avnet" H 2050 6700 60  0001 C CNN "Supplier"
 	1    18400 900
@@
 F 1 "10uf" H 19750 2550 50  0000 L CNN
 F 4 "603-CC603MRX5R5BB106" H 19700 2650 60  0001 C CNN "Mouser Part Number"
-F 5 "C0805C106M9PACTU" H 10300 3400 60  0001 C CNN "MPN"
+F 5 "08056D106MAT2A" H 10300 3400 60  0001 C CNN "MPN"
 F 6 "Avnet" H 10300 3400 60  0001 C CNN "Supplier"
 	1    19700 2650
@@
 P 10600 1050
 F 0 "C33" H 10650 1150 50  0000 L CNN
-F 1 ".1uF" H 10650 950 50  0000 L CNN
+F 1 "100nF" H 10650 950 50  0000 L CNN
 F 4 "581-060316C104K" H 10600 1050 60  0001 C CNN "Mouser Part Number"
 F 5 "C0603C104K3RAC7411" H 10600 1050 60  0001 C CNN "MPN"
@@
 P 8750 800
 F 0 "L3" V 8700 800 40  0000 C CNN
-F 1 "FB" V 8850 800 40  0000 C CNN
+F 1 "30ohmFB" V 8850 800 40  0000 C CNN
 F 4 "81-BLM21P300S" H 8750 800 60  0001 C CNN "Mouser Part Number"
 F 5 "BLM21PG300SN1D" V 5650 5750 60  0001 C CNN "MPN"
@@
 P 9350 1150
 F 0 "C29" H 9400 1250 50  0000 L CNN
-F 1 "10-100nF" H 9400 1050 50  0000 L CNN
+F 1 "100nF" H 9400 1050 50  0000 L CNN
 F 4 "581-060316C104K" H 9350 1150 60  0001 C CNN "Mouser Part Number"
-F 5 "12061C104KAT2A" H 2050 6700 60  0001 C CNN "MPN"
+F 5 "C0603C104K3RAC7411" H 2050 6700 60  0001 C CNN "MPN"
 F 6 "Avnet" H 2050 6700 60  0001 C CNN "Supplier"
 	1    9350 1150
@@
 P 7300 2250
 F 0 "C28" H 7350 2350 50  0000 L CNN
-F 1 "10-100nF" H 7350 2150 50  0000 L CNN
+F 1 "100nF" H 7350 2150 50  0000 L CNN
 F 4 "581-060316C104K" H 7300 2250 60  0001 C CNN "Mouser Part Number"
-F 5 "12061C104KAT2A" H 2050 6700 60  0001 C CNN "MPN"
+F 5 "C0603C104K3RAC7411" H 2050 6700 60  0001 C CNN "MPN"
 F 6 "Avnet" H 2050 6700 60  0001 C CNN "Supplier"
 	1    7300 2250
@@
 P 7050 3500
 F 0 "X1" H 7050 3650 60  0000 C CNN
-F 1 "15MHz" H 7050 3350 60  0000 C CNN
+F 1 "25MHz" H 7050 3350 60  0000 C CNN
 F 4 "815-ABM3C-25-D4YT" H 7050 3500 60  0001 C CNN "Mouser Part Number"
 F 5 "FQ5032B-25.000" H 7050 3500 60  0001 C CNN "MPN"
@@
 F 1 "10uF" H 10350 3300 50  0000 L CNN
 F 4 "603-CC603MRX5R5BB106" H 10300 3400 60  0001 C CNN "Mouser Part Number"
-F 5 "C0805C106M9PACTU" H 10300 3400 60  0001 C CNN "MPN"
+F 5 "08056D106MAT2A" H 10300 3400 60  0001 C CNN "MPN"
 F 6 "Avnet" H 10300 3400 60  0001 C CNN "Supplier"
 	1    10300 3400
@@
 P 15550 500
 F 0 "C27" H 15600 600 50  0000 L CNN
-F 1 ".1uF" H 15600 400 50  0000 L CNN
+F 1 "100nF" H 15600 400 50  0000 L CNN
 F 4 "581-060316C104K" H 15550 500 60  0001 C CNN "Mouser Part Number"
-F 5 "12061C104KAT2A" H 2050 6700 60  0001 C CNN "MPN"
+F 5 "C0603C104K3RAC7411" H 2050 6700 60  0001 C CNN "MPN"
 F 6 "Avnet" H 2050 6700 60  0001 C CNN "Supplier"
 	1    15550 500
@@
 F 4 "77-VJ0603Y332KXACBC" H 6800 5300 60  0001 C CNN "Mouser Part Number"
 F 5 "16V" H 6800 5300 60  0001 C CNN "Voltage"
-F 6 "C0603C332K5RACTU" H 5200 6300 60  0001 C CNN "MPN"
+F 6 "06035C332KAT2A" H 5200 6300 60  0001 C CNN "MPN"
 F 7 "Avnet" H 5200 6300 60  0001 C CNN "Supplier"
 	1    6800 5300
@@
 F 1 "3.3nF" H 5250 6200 50  0000 L CNN
 F 4 "77-VJ0603Y332KXACBC" H 5200 6300 60  0001 C CNN "Mouser Part Number"
-F 5 "16" H 5200 6300 60  0001 C CNN "Voltage"
-F 6 "C0603C332K5RACTU" H 5200 6300 60  0001 C CNN "MPN"
+F 5 "16V" H 5200 6300 60  0001 C CNN "Voltage"
+F 6 "06035C332KAT2A" H 5200 6300 60  0001 C CNN "MPN"
 F 7 "Avnet" H 5200 6300 60  0001 C CNN "Supplier"
 	1    5200 6300
@@
 F 2 "SM0603" H 550 6150 60  0001 C CNN
 F 4 "581-06031C102K" H 550 6150 60  0001 C CNN "Mouser Part Number"
-F 5 "100" H 550 6150 60  0001 C CNN "Voltage"
-F 6 "Avnet" H 1600 6700 60  0001 C CNN "Supplier"
+F 5 "Avnet" H 1600 6700 60  0001 C CNN "Supplier"
+F 6 "C0603C102K1RACTU" H 550 6150 60  0001 C CNN "MPN"
 	1    550  6150
 	1    0    0    -1
@@
 F 0 "R25" V 20980 5600 50  0000 C CNN
 F 1 "50" V 20900 5600 50  0000 C CNN
+F 4 "ERJ-3EKF51R0V " V 7100 1850 60  0001 C CNN "MPN"
+F 5 "Avnet" V 7100 1850 60  0001 C CNN "Supplier"
 	1    20900 5600
 	0    -1   -1   0
@@
 F 0 "R26" V 20980 5700 50  0000 C CNN
 F 1 "50" V 20900 5700 50  0000 C CNN
+F 4 "ERJ-3EKF51R0V " V 7100 1850 60  0001 C CNN "MPN"
+F 5 "Avnet" V 7100 1850 60  0001 C CNN "Supplier"
 	1    20900 5700
 	0    -1   -1   0
@@
 F 0 "R27" V 20980 5800 50  0000 C CNN
 F 1 "50" V 20900 5800 50  0000 C CNN
+F 4 "ERJ-3EKF51R0V " V 7100 1850 60  0001 C CNN "MPN"
+F 5 "Avnet" V 7100 1850 60  0001 C CNN "Supplier"
 	1    20900 5800
 	0    -1   -1   0
@@
 F 0 "R28" V 20980 5900 50  0000 C CNN
 F 1 "50" V 20900 5900 50  0000 C CNN
+F 4 "ERJ-3EKF51R0V " V 7100 1850 60  0001 C CNN "MPN"
+F 5 "Avnet" V 7100 1850 60  0001 C CNN "Supplier"
 	1    20900 5900
 	0    -1   -1   0
@@
 F 0 "R29" V 20980 6000 50  0000 C CNN
 F 1 "50" V 20900 6000 50  0000 C CNN
+F 4 "ERJ-3EKF51R0V " V 7100 1850 60  0001 C CNN "MPN"
+F 5 "Avnet" V 7100 1850 60  0001 C CNN "Supplier"
 	1    20900 6000
 	0    -1   -1   0
@@
 F 0 "R30" V 20980 6100 50  0000 C CNN
 F 1 "50" V 20900 6100 50  0000 C CNN
+F 4 "ERJ-3EKF51R0V " V 7100 1850 60  0001 C CNN "MPN"
+F 5 "Avnet" V 7100 1850 60  0001 C CNN "Supplier"
 	1    20900 6100
 	0    -1   -1   0
@@
 F 0 "R31" V 20980 6200 50  0000 C CNN
 F 1 "50" V 20900 6200 50  0000 C CNN
+F 4 "ERJ-3EKF51R0V " V 7100 1850 60  0001 C CNN "MPN"
+F 5 "Avnet" V 7100 1850 60  0001 C CNN "Supplier"
 	1    20900 6200
 	0    -1   -1   0
@@
 F 0 "R32" V 20980 6300 50  0000 C CNN
 F 1 "50" V 20900 6300 50  0000 C CNN
+F 4 "ERJ-3EKF51R0V " V 7100 1850 60  0001 C CNN "MPN"
+F 5 "Avnet" V 7100 1850 60  0001 C CNN "Supplier"
 	1    20900 6300
 	0    -1   -1   0
@@
 F 0 "R17" V 18780 5600 50  0000 C CNN
 F 1 "50" V 18700 5600 50  0000 C CNN
+F 4 "ERJ-3EKF51R0V " V 7100 1850 60  0001 C CNN "MPN"
+F 5 "Avnet" V 7100 1850 60  0001 C CNN "Supplier"
 	1    18700 5600
 	0    -1   -1   0
@@
 F 0 "R18" V 18780 5700 50  0000 C CNN
 F 1 "50" V 18700 5700 50  0000 C CNN
+F 4 "ERJ-3EKF51R0V " V 7100 1850 60  0001 C CNN "MPN"
+F 5 "Avnet" V 7100 1850 60  0001 C CNN "Supplier"
 	1    18700 5700
 	0    -1   -1   0
@@
 F 0 "R19" V 18780 5800 50  0000 C CNN
 F 1 "50" V 18700 5800 50  0000 C CNN
+F 4 "ERJ-3EKF51R0V " V 7100 1850 60  0001 C CNN "MPN"
+F 5 "Avnet" V 7100 1850 60  0001 C CNN "Supplier"
 	1    18700 5800
 	0    -1   -1   0
@@
 F 0 "R20" V 18780 5900 50  0000 C CNN
 F 1 "50" V 18700 5900 50  0000 C CNN
+F 4 "ERJ-3EKF51R0V " V 7100 1850 60  0001 C CNN "MPN"
+F 5 "Avnet" V 7100 1850 60  0001 C CNN "Supplier"
 	1    18700 5900
 	0    -1   -1   0
@@
 F 0 "R21" V 18780 6000 50  0000 C CNN
 F 1 "50" V 18700 6000 50  0000 C CNN
+F 4 "ERJ-3EKF51R0V " V 7100 1850 60  0001 C CNN "MPN"
+F 5 "Avnet" V 7100 1850 60  0001 C CNN "Supplier"
 	1    18700 6000
 	0    -1   -1   0
@@
 F 0 "R22" V 18780 6100 50  0000 C CNN
 F 1 "50" V 18700 6100 50  0000 C CNN
+F 4 "ERJ-3EKF51R0V " V 7100 1850 60  0001 C CNN "MPN"
+F 5 "Avnet" V 7100 1850 60  0001 C CNN "Supplier"
 	1    18700 6100
 	0    -1   -1   0
@@
 F 0 "R23" V 18780 6200 50  0000 C CNN
 F 1 "50" V 18700 6200 50  0000 C CNN
+F 4 "ERJ-3EKF51R0V " V 7100 1850 60  0001 C CNN "MPN"
+F 5 "Avnet" V 7100 1850 60  0001 C CNN "Supplier"
 	1    18700 6200
 	0    -1   -1   0
@@
 F 0 "R24" V 18780 6300 50  0000 C CNN
 F 1 "50" V 18700 6300 50  0000 C CNN
+F 4 "ERJ-3EKF51R0V " V 7100 1850 60  0001 C CNN "MPN"
+F 5 "Avnet" V 7100 1850 60  0001 C CNN "Supplier"
 	1    18700 6300
 	0    -1   -1   0
@@
 Text Label 21150 5700 0    60   ~ 0
 EXT_PB2
+$Comp
+L C C2
+U 1 1 512AE0F9
+P 20200 2650
+F 0 "C2" H 20250 2750 50  0000 L CNN
+F 1 "10uf" H 20250 2550 50  0000 L CNN
+F 4 "603-CC603MRX5R5BB106" H 20200 2650 60  0001 C CNN "Mouser Part Number"
+F 5 "08056D106MAT2A" H 10800 3400 60  0001 C CNN "MPN"
+F 6 "Avnet" H 10800 3400 60  0001 C CNN "Supplier"
+	1    20200 2650
+	1    0    0    -1
+$EndComp
 $EndSCHEMATC
